Commit message: whillの速度調節機能の追加

File: whill_description/urdf/whill_model_cr2.urdf (robot description, URDF)
Before this commit: robot whill_model_cr2, 12 links, 11 joints
Links:
- added link laser; collision cylinder length=0.03 radius=0.035; visual cylinder length=0.03 radius=0.035
- link base_link: geometry 
- link left_arm: geometry collision box size=0.09 0.07 0.535
- link right_arm: geometry collision box size=0.09 0.07 0.535
Joints:
- added joint laser_joint: type fixed, parent base_floor, child laser, origin xyz=0.40 0 0.30 rpy=0 0 0
- joint left_front_wheel_joint: axis 0 0 -1 -> 0 1 0; origin xyz=0.330 -0.235 0 rpy=-1.571 0 0 -> xyz=0.330 0.235 0 rpy=0 0 0
- joint left_wheel_joint: axis 0 0 1 -> 0 1 0; origin xyz=-0.3 0.260 0.015 rpy=1.571 0 0 -> xyz=-0.330 0.235 0 rpy=0 0 0
- joint right_front_wheel_joint: axis 0 0 1 -> 0 1 0; origin xyz=0.330 0.235 0 rpy=1.571 0 0 -> xyz=0.330 -0.235 0 rpy=0 0 0
- joint right_wheel_joint: axis 0 0 -1 -> 0 1 0; origin xyz=-0.3 -0.260 0.015 rpy=-1.571 0 0 -> xyz=-0.330 -0.235 0 rpy=0 0 0
